File: ecad/analog_switch_tester/analog_switch_tester/analog_switch_tester.kicad_pcb (KiCad board)
At the start: 2 copper layers, 30 x 30 mm, 10 parts, among them J1 Conn_01x03_Pin, U1 DRV5056A1xQDBZxR

Commit message: plot gerber files
Parts:
- added C10: 1uF, Capacitor_SMD:C_0603_1608Metric, F.Cu at (71.5, 69.0)
- added C11: 1uF, Capacitor_SMD:C_0603_1608Metric, F.Cu at (94.0, 67.8)
- added C12: 1uF, Capacitor_SMD:C_0603_1608Metric, F.Cu at (101.5, 69.0)
- added C13: 1uF, Capacitor_SMD:C_0603_1608Metric, F.Cu at (34.0, 97.8)
- added C14: 1uF, Capacitor_SMD:C_0603_1608Metric, F.Cu at (41.5, 99.0)
- added C15: 1uF, Capacitor_SMD:C_0603_1608Metric, F.Cu at (64.0, 97.8)
- added C16: 1uF, Capacitor_SMD:C_0603_1608Metric, F.Cu at (71.5, 99.0)
- added C17: 1uF, Capacitor_SMD:C_0603_1608Metric, F.Cu at (94.0, 97.8)
- added C18: 1uF, Capacitor_SMD:C_0603_1608Metric, F.Cu at (101.5, 99.0)
- added C3: 1uF, Capacitor_SMD:C_0603_1608Metric, F.Cu at (64.0, 37.8)
- added C4: 1uF, Capacitor_SMD:C_0603_1608Metric, F.Cu at (71.5, 39.0)
- added C5: 1uF, Capacitor_SMD:C_0603_1608Metric, F.Cu at (94.0, 37.8)
- added C6: 1uF, Capacitor_SMD:C_0603_1608Metric, F.Cu at (101.5, 39.0)
- added C7: 1uF, Capacitor_SMD:C_0603_1608Metric, F.Cu at (34.0, 67.8)
- added C8: 1uF, Capacitor_SMD:C_0603_1608Metric, F.Cu at (41.5, 69.0)
- added C9: 1uF, Capacitor_SMD:C_0603_1608Metric, F.Cu at (64.0, 67.8)
- added J2: Conn_01x03_Pin, Connector_PinHeader_2.54mm:PinHeader_1x03_P2.54mm_Vertical, F.Cu at (68.4, 46.6)
- added J3: Conn_01x03_Pin, Connector_PinHeader_2.54mm:PinHeader_1x03_P2.54mm_Vertical, F.Cu at (98.4, 46.6)
- added J4: Conn_01x03_Pin, Connector_PinHeader_2.54mm:PinHeader_1x03_P2.54mm_Vertical, F.Cu at (38.4, 76.6)
- added J5: Conn_01x03_Pin, Connector_PinHeader_2.54mm:PinHeader_1x03_P2.54mm_Vertical, F.Cu at (68.4, 76.6)
- added J6: Conn_01x03_Pin, Connector_PinHeader_2.54mm:PinHeader_1x03_P2.54mm_Vertical, F.Cu at (98.4, 76.6)
- added J7: Conn_01x03_Pin, Connector_PinHeader_2.54mm:PinHeader_1x03_P2.54mm_Vertical, F.Cu at (38.4, 106.6)
- added J8: Conn_01x03_Pin, Connector_PinHeader_2.54mm:PinHeader_1x03_P2.54mm_Vertical, F.Cu at (68.4, 106.6)
- added J9: Conn_01x03_Pin, Connector_PinHeader_2.54mm:PinHeader_1x03_P2.54mm_Vertical, F.Cu at (98.4, 106.6)
- added MB_10: MountingHole_3.2mm_M3, MountingHole:MountingHole_3.2mm_M3, F.Cu at (106.8, 22.9)
- added MB_11: MountingHole_3.2mm_M3, MountingHole:MountingHole_3.2mm_M3, F.Cu at (84.8, 44.9)
- added MB_12: MountingHole_3.2mm_M3, MountingHole:MountingHole_3.2mm_M3, F.Cu at (106.8, 44.9)
- added MB_13: MountingHole_3.2mm_M3, MountingHole:MountingHole_3.2mm_M3, F.Cu at (24.8, 52.9)
- added MB_14: MountingHole_3.2mm_M3, MountingHole:MountingHole_3.2mm_M3, F.Cu at (46.8, 52.9)
- added MB_15: MountingHole_3.2mm_M3, MountingHole:MountingHole_3.2mm_M3, F.Cu at (24.8, 74.9)
- added MB_16: MountingHole_3.2mm_M3, MountingHole:MountingHole_3.2mm_M3, F.Cu at (46.8, 74.9)
- added MB_17: MountingHole_3.2mm_M3, MountingHole:MountingHole_3.2mm_M3, F.Cu at (54.8, 52.9)
- added MB_18: MountingHole_3.2mm_M3, MountingHole:MountingHole_3.2mm_M3, F.Cu at (76.8, 52.9)
- added MB_19: MountingHole_3.2mm_M3, MountingHole:MountingHole_3.2mm_M3, F.Cu at (54.8, 74.9)
- added MB_20: MountingHole_3.2mm_M3, MountingHole:MountingHole_3.2mm_M3, F.Cu at (76.8, 74.9)
- added MB_21: MountingHole_3.2mm_M3, MountingHole:MountingHole_3.2mm_M3, F.Cu at (84.8, 52.9)
- added MB_22: MountingHole_3.2mm_M3, MountingHole:MountingHole_3.2mm_M3, F.Cu at (106.8, 52.9)
- added MB_23: MountingHole_3.2mm_M3, MountingHole:MountingHole_3.2mm_M3, F.Cu at (84.8, 74.9)
- added MB_24: MountingHole_3.2mm_M3, MountingHole:MountingHole_3.2mm_M3, F.Cu at (106.8, 74.9)
- added MB_25: MountingHole_3.2mm_M3, MountingHole:MountingHole_3.2mm_M3, F.Cu at (24.8, 82.9)
- added MB_26: MountingHole_3.2mm_M3, MountingHole:MountingHole_3.2mm_M3, F.Cu at (46.8, 82.9)
- added MB_27: MountingHole_3.2mm_M3, MountingHole:MountingHole_3.2mm_M3, F.Cu at (24.8, 104.9)
- added MB_28: MountingHole_3.2mm_M3, MountingHole:MountingHole_3.2mm_M3, F.Cu at (46.8, 104.9)
- added MB_29: MountingHole_3.2mm_M3, MountingHole:MountingHole_3.2mm_M3, F.Cu at (54.8, 82.9)
- added MB_30: MountingHole_3.2mm_M3, MountingHole:MountingHole_3.2mm_M3, F.Cu at (76.8, 82.9)
- added MB_31: MountingHole_3.2mm_M3, MountingHole:MountingHole_3.2mm_M3, F.Cu at (54.8, 104.9)
- added MB_32: MountingHole_3.2mm_M3, MountingHole:MountingHole_3.2mm_M3, F.Cu at (76.8, 104.9)
- added MB_33: MountingHole_3.2mm_M3, MountingHole:MountingHole_3.2mm_M3, F.Cu at (84.8, 82.9)
- added MB_34: MountingHole_3.2mm_M3, MountingHole:MountingHole_3.2mm_M3, F.Cu at (106.8, 82.9)
- added MB_35: MountingHole_3.2mm_M3, MountingHole:MountingHole_3.2mm_M3, F.Cu at (84.8, 104.9)
- added MB_36: MountingHole_3.2mm_M3, MountingHole:MountingHole_3.2mm_M3, F.Cu at (106.8, 104.9)
- added MB_5: MountingHole_3.2mm_M3, MountingHole:MountingHole_3.2mm_M3, F.Cu at (54.8, 22.9)
- added MB_6: MountingHole_3.2mm_M3, MountingHole:MountingHole_3.2mm_M3, F.Cu at (76.8, 22.9)
- added MB_7: MountingHole_3.2mm_M3, MountingHole:MountingHole_3.2mm_M3, F.Cu at (54.8, 44.9)
- added MB_8: MountingHole_3.2mm_M3, MountingHole:MountingHole_3.2mm_M3, F.Cu at (76.8, 44.9)
- added MB_9: MountingHole_3.2mm_M3, MountingHole:MountingHole_3.2mm_M3, F.Cu at (84.8, 22.9)
- added Mount2: Conn_01x03_Pin, Connector_PinHeader_2.54mm:PinHeader_1x03_P2.54mm_Vertical, F.Cu at (63.3, 21.2)
- added Mount3: Conn_01x03_Pin, Connector_PinHeader_2.54mm:PinHeader_1x03_P2.54mm_Vertical, F.Cu at (93.3, 21.2)
- added Mount4: Conn_01x03_Pin, Connector_PinHeader_2.54mm:PinHeader_1x03_P2.54mm_Vertical, F.Cu at (33.3, 51.2)
- added Mount5: Conn_01x03_Pin, Connector_PinHeader_2.54mm:PinHeader_1x03_P2.54mm_Vertical, F.Cu at (63.3, 51.2)
- added Mount6: Conn_01x03_Pin, Connector_PinHeader_2.54mm:PinHeader_1x03_P2.54mm_Vertical, F.Cu at (93.3, 51.2)
- added Mount7: Conn_01x03_Pin, Connector_PinHeader_2.54mm:PinHeader_1x03_P2.54mm_Vertical, F.Cu at (33.3, 81.2)
- added Mount8: Conn_01x03_Pin, Connector_PinHeader_2.54mm:PinHeader_1x03_P2.54mm_Vertical, F.Cu at (63.3, 81.2)
- added Mount9: Conn_01x03_Pin, Connector_PinHeader_2.54mm:PinHeader_1x03_P2.54mm_Vertical, F.Cu at (93.3, 81.2)
- added R2: 100, Resistor_SMD:R_0603_1608Metric, F.Cu at (69.0, 38.9)
- added R3: 100, Resistor_SMD:R_0603_1608Metric, F.Cu at (99.0, 38.9)
- added R4: 100, Resistor_SMD:R_0603_1608Metric, F.Cu at (39.0, 68.9)
- added R5: 100, Resistor_SMD:R_0603_1608Metric, F.Cu at (69.0, 68.9)
- added R6: 100, Resistor_SMD:R_0603_1608Metric, F.Cu at (99.0, 68.9)
- added R7: 100, Resistor_SMD:R_0603_1608Metric, F.Cu at (39.0, 98.9)
- added R8: 100, Resistor_SMD:R_0603_1608Metric, F.Cu at (69.0, 98.9)
- added R9: 100, Resistor_SMD:R_0603_1608Metric, F.Cu at (99.0, 98.9)
- added U2: DRV5056A1xQDBZxR, Udong:SW_Cherry_MX_PCB_1.00u_hall_effect, F.Cu at (65.8, 33.9)
- added U3: DRV5056A1xQDBZxR, Udong:SW_Cherry_MX_PCB_1.00u_hall_effect, F.Cu at (95.8, 33.9)
- added U4: DRV5056A1xQDBZxR, Udong:SW_Cherry_MX_PCB_1.00u_hall_effect, F.Cu at (35.8, 63.9)
- added U5: DRV5056A1xQDBZxR, Udong:SW_Cherry_MX_PCB_1.00u_hall_effect, F.Cu at (65.8, 63.9)
- added U6: DRV5056A1xQDBZxR, Udong:SW_Cherry_MX_PCB_1.00u_hall_effect, F.Cu at (95.8, 63.9)
- added U7: DRV5056A1xQDBZxR, Udong:SW_Cherry_MX_PCB_1.00u_hall_effect, F.Cu at (35.8, 93.9)
- added U8: DRV5056A1xQDBZxR, Udong:SW_Cherry_MX_PCB_1.00u_hall_effect, F.Cu at (65.8, 93.9)
- added U9: DRV5056A1xQDBZxR, Udong:SW_Cherry_MX_PCB_1.00u_hall_effect, F.Cu at (95.8, 93.9)
Routing:
- net GNDA: track 26.9 -> 242.5 mm
- net OUT: track 13.8 -> 124.3 mm
- net V_AREF: track 12.9 -> 116.3 mm
- net Net-(U1-OUT): track 6.30 -> 56.7 mm
Other:
- board size 30 x 30 mm -> 90 x 90 mm
- board text added: "< V-CUT"
- board text added: "V-CUT >"

Commit message: .
Parts:
- removed C10, C11, C12, C13, C14, C15, C16, C17, C18, C3, C4, C5, C6, C7, C8, C9: 1uF, Capacitor_SMD:C_0603_1608Metric
- removed J2, J3, J4, J5, J6, J7, J8, J9, Mount2, Mount3, Mount4, Mount5, Mount6, Mount7, Mount8, Mount9: Conn_01x03_Pin, Connector_PinHeader_2.54mm:PinHeader_1x03_P2.54mm_Vertical
- removed MB_10, MB_11, MB_12, MB_13, MB_14, MB_15, MB_16, MB_17, MB_18, MB_19, MB_20, MB_21, MB_22, MB_23, MB_24, MB_25, MB_26, MB_27, MB_28, MB_29, MB_30, MB_31, MB_32, MB_33, MB_34, MB_35, MB_36, MB_5, MB_6, MB_7, MB_8, MB_9: MountingHole_3.2mm_M3, MountingHole:MountingHole_3.2mm_M3
- removed R2, R3, R4, R5, R6, R7, R8, R9: 100, Resistor_SMD:R_0603_1608Metric
- removed U2, U3, U4, U5, U6, U7, U8, U9: DRV5056A1xQDBZxR, Udong:SW_Cherry_MX_PCB_1.00u_hall_effect
- moved C2 2.67 mm to (38.9, 38.8), turned to -90 degrees
- moved R1 2.41 mm to (41.4, 38.9), turned to -90 degrees
Routing:
- net GNDA: track 242.5 -> 23.2 mm
- net OUT: track 124.3 -> 8.40 mm
- net V_AREF: track 116.3 -> 12.9 mm
- net Net-(U1-OUT): track 56.7 -> 9.18 mm
Other:
- board size 90 x 90 mm -> 30 x 30 mm
- board text added: "It might be a nice idea to rotate the center 90 degrees so that we can split GND/VCC and OUT to different side of the component. (connections have to avoid tiny holes for key switches) GND--+---------C | | C--- U ---R----OUT VCC--+"
- board text removed: "< V-CUT"
- board text removed: "V-CUT >"
