File: ecad/mainboard/digital_switches.kicad_sch (KiCad schematic)
At the start: 1 part, among them J1 Conn_01x02_Socket

Commit message: place parts except analog switches
Parts:
- removed J1: Conn_01x02_Socket, symbol Connector:Conn_01x02_Socket
Changed lines of the file:
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@@
 	(generator_version "8.0")
 	(paper "A4")
-	(symbol
-		(lib_id "Connector:Conn_01x02_Socket")
-		(at 152.4 110.49 0)
-		(unit 1)
-		(exclude_from_sim no)
-		(in_bom yes)
-		(on_board yes)
-		(dnp no)
-		(fields_autoplaced yes)
-		(property "Reference" "J1"
-			(at 153.67 110.4899 0)
-			(effects
-				(font
-					(size 1.27 1.27)
-				)
-				(justify left)
-			)
-		)
-		(property "Value" "Conn_01x02_Socket"
-			(at 153.67 113.0299 0)
-			(effects
-				(font
-					(size 1.27 1.27)
-				)
-				(justify left)
-			)
-		)
-		(property "Footprint" ""
-			(at 152.4 110.49 0)
-			(effects
-				(font
-					(size 1.27 1.27)
-				)
-				(hide yes)
-			)
-		)
-		(property "Datasheet" "~"
-			(at 152.4 110.49 0)
-			(effects
-				(font
-					(size 1.27 1.27)
-				)
-				(hide yes)
-			)
-		)
-		(property "Description" "Generic connector, single row, 01x02, script generated"
-			(at 152.4 110.49 0)
-			(effects
-				(font
-					(size 1.27 1.27)
-				)
-				(hide yes)
-			)
-		)
-		(pin "2"
-		)
-		(pin "1"
-		)
-		(instances
-			(project ""
-				(path "/b1313647-8d60-4294-add7-71c03651cfe3/89bd7dd7-1036-4268-8ed9-187e101d08a4"
-					(reference "J1")
-					(unit 1)
-				)
-			)
-		)
-	)
 )
