File: ecad/mainboard/mainboard.kicad_pcb (KiCad board)
At the start: 2 copper layers, 117 parts, among them J1 TYPE-C-31-M-12, J2 SWD, J3 UART, SW1 BOOTSEL, SW2 RUN, SW3 Key_Switch_with_LED, SW4 Key_Switch_with_LED, U1 NCP1117-3.3_SOT223, U10 DRV5056A3xQDBZxR, U11 DRV5056A3xQDBZxR, U12 DRV5056A3xQDBZxR, U13 DRV5056A3xQDBZxR, U14 DRV5056A3xQDBZxR, U15 DRV5056A3xQDBZxR, U16 DRV5056A3xQDBZxR, U17 DRV5056A3xQDBZxR, U18 DRV5056A3xQDBZxR, U19 DRV5056A3xQDBZxR, U2 USBLC6-2SC6, U20 DRV5056A3xQDBZxR, U21 DRV5056A3xQDBZxR, U22 CD4051BM96, U23 CD4051BM96, U3 W25Q128JVS, U4 74AHCT1G125, U5 RP2040, U6 DRV5056A3xQDBZxR, U7 DRV5056A3xQDBZxR, U8 DRV5056A3xQDBZxR, U9 DRV5056A3xQDBZxR, Y1 ABM8-272-T3

Commit message: .
Parts:
- U10, U11, U12, U13, U14, U15, U16, U17, U18, U19, U20, U21, U6, U7, U8, U9: footprint Package_TO_SOT_SMD:SOT-23 -> Udong:SW_Cherry_MX_PCB_1.00u_hall_effect
- moved U6 124.3 mm to (54.2, 145.9)
- moved U7 94.8 mm to (86.7, 143.6)
- moved U8 89.9 mm to (103.4, 127.1)
- moved R24 82.3 mm to (305.7, 214.1)
- moved R25 82.3 mm to (305.7, 216.6)
- moved R27 82.3 mm to (305.7, 221.6)
- moved R28 82.3 mm to (305.7, 224.1)
- moved R23 82.3 mm to (305.7, 211.6)
- moved R26 82.3 mm to (305.7, 219.1)
- moved R29 82.3 mm to (305.7, 226.6)
- moved C38 77.5 mm to (247.5, 124.7), turned to 180 degrees
- moved U9 73.7 mm to (113.8, 145.3)
- moved U14 67.3 mm to (249.4, 130.7)
- moved C37 58.4 mm to (250.2, 135.6)
- moved U17 51.1 mm to (336.7, 130.3)
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- renumbered C25 to C22, C22 to C23, C26 to C24, C23 to C25, C27 to C26, C24 to C27, C33 to C30, C30 to C31, C34 to C32, C31 to C33, C35 to C34, C32 to C35, C41 to C38, C38 to C39, C42 to C40, C39 to C41, C43 to C42, C40 to C43, C49 to C46, C46 to C47, C50 to C48, C47 to C49, C51 to C50, C48 to C51

Commit message: place all parts
Parts:
- moved H3 387.6 mm to (375.0, 235.0)
- moved H4 341.4 mm to (375.0, 25.0)
- moved H2 193.3 mm to (45.0, 235.0)
- moved C44 173.0 mm to (278.6, 51.5), turned to 180 degrees
- moved R25 165.3 mm to (278.6, 53.5), turned to 180 degrees
- moved R24 156.2 mm to (203.5, 96.0), turned to 180 degrees
- moved C43 156.0 mm to (281.6, 62.0)
- moved C28 155.0 mm to (173.5, 84.0), turned to 180 degrees
- moved R16 145.7 mm to (83.5, 91.0), turned to 180 degrees
- moved R17 144.9 mm to (173.4, 86.0), turned to 180 degrees
- moved C27 141.6 mm to (176.5, 94.5)
- moved R26 139.5 mm to (188.5, 143.5), turned to 180 degrees
- moved R15 139.1 mm to (113.5, 86.0), turned to 180 degrees
- moved R14 138.8 mm to (143.4, 81.0), turned to 180 degrees
- moved C42 133.3 mm to (203.6, 94.0), turned to 180 degrees
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
Commit message: .
Parts:
- moved J2 0.27 mm to (174.3, 23.2)
Other:
- board outline added: 340 x 220 mm
Changed lines of the file:
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@@
 	(footprint "Connector_JST:JST_SH_BM03B-SRSS-TB_1x03-1MP_P1.00mm_Vertical"
 		(layer "F.Cu")
-		(at 174.312 23.447)
+		(at 174.312 23.175)
 		(descr "JST SH series connector, BM03B-SRSS-TB (http://www.jst-mfg.com/product/pdf/eng/eSH.pdf), generated with kicad-footprint-generator")
 		(tags "connector JST SH vertical")
@@
 		(net 4)
 	)
+	(gr_rect
+		(start 40 20)
+		(end 380 240)
+		(stroke
+			(width 0.05)
+			(type default)
+		)
+		(fill none)
+		(layer "Edge.Cuts")
+	)
 	(gr_line
