File: ecad/mainboard/mainboard.kicad_pcb (KiCad board)
At the start: 2 copper layers, 340 x 220 mm, 117 parts, among them J1 TYPE-C-31-M-12, J2 SWD, J3 UART, SW1 BOOTSEL, SW2 RUN, SW3 Key_Switch_with_LED, SW4 Key_Switch_with_LED, U1 NCP1117-3.3_SOT223, U10 DRV5056A3xQDBZxR, U11 DRV5056A3xQDBZxR, U12 DRV5056A3xQDBZxR, U13 DRV5056A3xQDBZxR, U14 DRV5056A3xQDBZxR, U15 DRV5056A3xQDBZxR, U16 DRV5056A3xQDBZxR, U17 DRV5056A3xQDBZxR, U18 DRV5056A3xQDBZxR, U19 DRV5056A3xQDBZxR, U2 USBLC6-2SC6, U20 DRV5056A3xQDBZxR, U21 DRV5056A3xQDBZxR, U22 CD4051BM96, U23 CD4051BM96, U3 W25Q128JVS, U4 74AHCT1G125, U5 RP2040, U6 DRV5056A3xQDBZxR, U7 DRV5056A3xQDBZxR, U8 DRV5056A3xQDBZxR, U9 DRV5056A3xQDBZxR, Y1 ABM8-272-T3

Commit message: fix all DRC errors for connected parts
Parts:
- R1: value R -> 220k
- R4: value R -> 40k
- U5: footprint Package_DFN_QFN:QFN-56-1EP_7x7mm_P0.4mm_EP3.2x3.2mm_ThermalVias -> Udong:RP2040-QFN-56
- moved C51 92.1 mm to (281.3, 92.2)
- moved R29 92.1 mm to (278.3, 83.5)
- moved C52 91.9 mm to (278.3, 81.8)
- moved R28 88.8 mm to (248.2, 93.0)
- moved C49 88.7 mm to (251.4, 102.2)
- moved C50 88.7 mm to (248.4, 91.5)
- moved C20 80.9 mm to (345.1, 78.5)
- moved C40 78.3 mm to (188.5, 141.8)
- moved C39 78.1 mm to (191.5, 152.0)
- moved R23 78.1 mm to (188.4, 143.5)
- moved U15 78.1 mm to (189.9, 147.5)
- moved U20 67.0 mm to (249.9, 97.5)
- moved C37 65.1 mm to (336.4, 127.0)
- moved C38 65.1 mm to (333.4, 116.8)
- moved R22 65.1 mm to (333.5, 118.6)
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Connections:
- J3 pad 1: UART_RX -> UART_TX
- J3 pad 3: UART_TX -> UART_RX
Routing:
- net DS_0_IN: track 0.00 -> 227.6 mm
- net GND: track 0.00 -> 168.1 mm, vias 0 -> 34
- net AS4: track 0.00 -> 153.2 mm
- net AS8: track 0.00 -> 144.6 mm
- net +3.3V: track 0.00 -> 143.6 mm, vias 0 -> 38
- net AS2: track 0.00 -> 139.7 mm
- net AS6: track 0.00 -> 126.0 mm
- net AS1: track 0.00 -> 108.6 mm
- net LED_OUT_5V: track 0.00 -> 94.8 mm
- net AS7: track 0.00 -> 94.0 mm
- net AS13: track 0.00 -> 93.5 mm
- net AS9: track 0.00 -> 92.7 mm
- net SWCLK: track 0.00 -> 89.9 mm
- net AS12: track 0.00 -> 84.2 mm
- net AS0: track 0.00 -> 78.6 mm
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- added copper zone on F.Cu, net +3.3V
- added copper zone on In2.Cu, net +3.3V
- added copper zone on B.Cu, net GND
- added copper zone on F.Cu, net GND
- added copper zone on In1.Cu, net GND
- added copper zone on F.Cu, net VBUS
- added copper zone on In2.Cu, net VBUS
Other:
- copper layers 2 -> 4

Commit message: refactor some patterns
Parts:
- added H10: MountingHole, MountingHole:MountingHole_2.7mm_M2.5, F.Cu at (210.0, 230.0)
- added H5: MountingHole, MountingHole:MountingHole_2.7mm_M2.5, F.Cu at (135.0, 30.0)
- added H6: MountingHole, MountingHole:MountingHole_2.7mm_M2.5, F.Cu at (285.0, 30.0)
- added H7: MountingHole, MountingHole:MountingHole_2.7mm_M2.5, F.Cu at (285.0, 160.0)
- added H8: MountingHole, MountingHole:MountingHole_2.7mm_M2.5, F.Cu at (135.0, 160.0)
- added H9: MountingHole, MountingHole:MountingHole_2.7mm_M2.5, F.Cu at (210.0, 130.0)
- moved C20 210.1 mm to (135.8, 60.1)
- moved H1 7.07 mm to (50.0, 30.0)
- moved H2 7.07 mm to (50.0, 230.0)
- moved H3 7.07 mm to (370.0, 230.0)
- moved H4 7.07 mm to (370.0, 30.0)
- moved C4 0.44 mm to (208.5, 42.6)
- moved C10 0.32 mm to (216.4, 51.9)
- moved C6 0.30 mm to (209.5, 42.9)
Routing:
- net +3.3V: track 143.6 -> 130.8 mm, vias 38 -> 40
- net GND: track 168.1 -> 159.6 mm, vias 34 -> 54
- net DS_0_IN: track 227.6 -> 219.9 mm
- net DS_1_IN: track 78.6 -> 72.7 mm
- net AS9: track 92.7 -> 97.8 mm
- net +1V1: track 20.6 -> 15.5 mm
- net VBUS: track 38.5 -> 37.3 mm
- net SWCLK: track 89.9 -> 88.8 mm
- net AS3: track 50.8 -> 49.9 mm
- net AS0: track 78.6 -> 78.0 mm
- net MUX0_OUT: track 28.5 -> 27.9 mm
- net Net-(U17-OUT): track 3.41 -> 2.91 mm
- net UART_TX: track 48.6 -> 48.1 mm
- added copper zone on F.Cu, net +1V1

Commit message: .
Parts:
- moved U22 0.06 mm to (212.5, 69.5)
Routing:
- net RUN: track 40.5 -> 58.5 mm
- net SWD: track 76.9 -> 92.7 mm
- net DS_1_IN: track 72.7 -> 83.5 mm
- net AS10: track 38.6 -> 47.2 mm
- net AS9: track 97.8 -> 91.9 mm
- net GND: track 159.6 -> 164.9 mm, vias 54 -> 55
- net DS_0_IN: track 219.9 -> 215.1 mm
- net AS7: track 93.9 -> 91.0 mm
- net AS4: track 153.1 -> 150.9 mm
- net AS5: track 68.3 -> 66.9 mm
- net +3.3V: track 130.8 -> 129.5 mm, vias 40 -> 41
- net SWCLK: track 88.8 -> 87.5 mm
- net AS6: track 125.8 -> 124.5 mm
- net Net-(U15-OUT): track 3.38 -> 2.82 mm
- net Net-(U9-OUT): track 3.38 -> 2.82 mm
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- added copper zone on In2.Cu, net GND

Commit message: Udong board rev.1
Parts:
- removed R6: 0, Resistor_SMD:R_0402_1005Metric
- moved C35 1.43 mm to (145.8, 123.1)
- moved C33 1.40 mm to (115.7, 128.1)
- moved C23 1.40 mm to (115.7, 95.7)
- moved C21 1.37 mm to (145.7, 90.6)
- moved C27 1.27 mm to (175.7, 95.5)
- moved C29 1.27 mm to (85.7, 133.0)
- moved C25 1.18 mm to (85.8, 100.4)
- moved C39 1.16 mm to (190.7, 152.8)
- moved C43 1.03 mm to (280.9, 62.7)
- moved C45 1.02 mm to (220.8, 162.6)
- moved C37 1.02 mm to (335.6, 127.6)
- moved C47 1.00 mm to (310.7, 102.4)
- moved C49 1.00 mm to (250.6, 102.9)
- moved C31 0.98 mm to (175.7, 127.6)
- moved C41 0.90 mm to (205.8, 105.2)
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Connections:
- U5 pad 11: GPIO_UNUSED -> GND
- U5 pad 12: GPIO_UNUSED -> GND
- U5 pad 13: GPIO_UNUSED -> GND
- U5 pad 14: GPIO_UNUSED -> GND
- U5 pad 15: GPIO_UNUSED -> GND
- U5 pad 16: GPIO_UNUSED -> GND
- U5 pad 17: GPIO_UNUSED -> GND
- U5 pad 18: GPIO_UNUSED -> GND
- U5 pad 4: GPIO_UNUSED -> GND
- U5 pad 40: GPIO_UNUSED -> GND
- U5 pad 41: GPIO_UNUSED -> GND
- U5 pad 5: GPIO_UNUSED -> GND
- U5 pad 7: GPIO_UNUSED -> GND
- U5 pad 8: GPIO_UNUSED -> GND
- U5 pad 9: GPIO_UNUSED -> GND
Routing:
- net GND: track 164.9 -> 157.0 mm, vias 55 -> 50
- net QSPI_SS: track 22.3 -> 29.8 mm
- net +3.3V: track 129.5 -> 126.5 mm, vias 41 -> 42
- net VBUS: track 37.3 -> 35.0 mm, vias 4 -> 5
- net SHIELD: track 36.2 -> 37.7 mm
Other:
- board text added: "Udong Board rev.1"

Commit message: .
Changed lines of the file:
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@@
 			(disableapertmacros no)
 			(usegerberextensions no)
-			(usegerberattributes yes)
+			(usegerberattributes no)
 			(usegerberadvancedattributes yes)
 			(creategerberjobfile yes)
@@
 			(outputformat 1)
 			(mirror no)
-			(drillshape 1)
+			(drillshape 0)
 			(scaleselection 1)
-			(outputdirectory "")
+			(outputdirectory "gerber/")
 		)
 	)
@@
 		(fp_arc
 			(start 5.436 16.231)
-			(mid 4.002296 15.679932)
+			(mid 4.002293 15.679933)
 			(end 3.277 14.326)
 			(stroke

Commit message: add new footprints but broken pcb
Parts:
- added D2: SK6812MINI, Udong:MX_Socket_LED, F.Cu at (339.7, 47.2)
- added D3: SK6812MINI, Udong:MX_Socket_LED, F.Cu at (362.2, 47.2)
- D1: footprint LED_SMD:LED_0603_1608Metric -> LED_SMD:LED_0805_2012Metric
- SW1: value BOOTSEL -> TS-1187A-B-A-B
- SW2: value RUN -> TS-1187A-B-A-B
- SW3: value Key_Switch_with_LED -> Digital_Switch_1; footprint geek_rabb1t:MX_Socket_LED -> Udong:MX_Socket
- SW4: value Key_Switch_with_LED -> Digital_Switch_2; footprint geek_rabb1t:MX_Socket_LED -> Udong:MX_Socket
- U1: value NCP1117-3.3_SOT223 -> NCP1117ST33T3G
Connections:
- R12 pad 2: Net-(SW3-DIN) -> Net-(D2-DIN)
- SW3 pad 1: DS_0_IN -> GND
- SW3 pad 2: GND -> DS_0_IN
- SW4 pad 1: DS_1_IN -> GND
- SW4 pad 2: GND -> DS_1_IN
Routing:
- net Net-(SW3-DOUT): track 17.6 -> 0.00 mm
- net Net-(D2-DOUT): track 0.00 -> 17.6 mm
- net Net-(SW3-DIN): track 2.20 -> 0.00 mm
- net Net-(D2-DIN): track 0.00 -> 2.20 mm
- net +3.3V: vias 42 -> 41

Commit message: .
Parts:
- R9: value DNF -> 0
- SW3: value Digital_Switch_1 -> SW_Push
- SW4: value Digital_Switch_2 -> SW_Push
- moved R9 0.07 mm to (197.0, 31.6)
- moved D2 0.05 mm to (339.8, 47.2)
Connections:
- R9 pad 1: +3.3V -> QSPI_SS
- R9 pad 2: QSPI_SS -> +3.3V
- SW3 pad 1: GND -> DS_0_IN
- SW3 pad 2: DS_0_IN -> GND
- SW4 pad 1: GND -> DS_1_IN
- SW4 pad 2: DS_1_IN -> GND
Routing:
- net +3.3V: vias 41 -> 42

Commit message: rev1.1
Parts:
- removed R9: 0, Resistor_SMD:R_0402_1005Metric
- moved C15 10.9 mm to (206.1, 36.6), turned to 90 degrees
- moved R8 0.40 mm to (225.8, 38.8)
Routing:
- net +3.3V: track 126.5 -> 124.8 mm, vias 42 -> 41
- net SHIELD: track 37.7 -> 36.1 mm
- net QSPI_SS: track 29.8 -> 28.4 mm
- net GND: track 157.0 -> 156.2 mm
