File: ecad/mainboard_top_plate/mainboard_top_plate.kicad_pcb (KiCad board)
At the start: 2 copper layers, 340 x 220 mm, 28 parts, among them SW3 SW_Push, SW4 SW_Push, U10 DRV5056A3xQDBZxR, U11 DRV5056A3xQDBZxR, U12 DRV5056A3xQDBZxR, U13 DRV5056A3xQDBZxR, U14 DRV5056A3xQDBZxR, U15 DRV5056A3xQDBZxR, U16 DRV5056A3xQDBZxR, U17 DRV5056A3xQDBZxR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

Commit message: rev2 board
Parts:
- removed H10, H6, H7, H8, H9: MountingHole, MountingHole:MountingHole_2.7mm_M2.5
- added ?: , , F.Cu at (221.0, 44.0)
- added REF**: MountingHole_3.7mm, MountingHole:MountingHole_3.7mm, F.Cu at (60.0, 50.0)
- added REF**: MountingHole_3.7mm, MountingHole:MountingHole_3.7mm, F.Cu at (360.0, 260.0)
- added REF**: MountingHole_3.7mm, MountingHole:MountingHole_3.7mm, F.Cu at (60.0, 260.0)
- added REF**: MountingHole_3.7mm, MountingHole:MountingHole_3.7mm, F.Cu at (360.0, 50.0)
- H1, H2, H3, H4, H5: value MountingHole -> MountingHole_Pad; footprint MountingHole:MountingHole_2.7mm_M2.5 -> MountingHole:MountingHole_3.7mm_Pad_Via
- moved H2 297.7 mm to (280.0, 70.0)
- moved H4 246.1 mm to (140.0, 160.0)
- moved H5 214.1 mm to (280.0, 160.0)
- moved U19 205.6 mm to (88.0, 146.0)
- moved SW4 181.1 mm to (176.0, 130.0)
- moved H3 168.0 mm to (210.0, 130.0)
- moved U14 166.3 mm to (146.0, 128.0)
- moved U8 143.3 mm to (204.0, 112.0)
- moved U9 127.9 mm to (280.0, 90.0)
- moved H1 120.7 mm to (140.0, 70.0)
- moved U18 120.1 mm to (116.0, 66.0)
- moved U17 117.7 mm to (336.0, 142.0)
- moved U10 117.0 mm to (176.0, 98.0)
- moved U21 100.5 mm to (220.0, 178.0)
- moved U11 97.9 mm to (250.0, 118.0)
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Other:
- board size 340 x 220 mm -> 320 x 230 mm
- board text added: "Udong Board rev.2"
- board text removed: "Udong Board rev.1"

Commit message: Hardware version 1.0
Parts:
- added G***: LOGO, Udong:udong_logo, F.Cu at (97.0, 247.5)
Other:
- board text added: "Board ver.1.0"
- board text removed: "Udong Board rev.2"
